Commit message: stage rearrange

File: src/ackermann_car_description/urdf/ackermann_car.urdf.xacro (robot description, xacro)
@@ -53,5 +53,5 @@
         <origin xyz="0 0 0" rpy="${pi/2} 0 0"/>
         <geometry><cylinder radius="${wheel_r}" length="${wheel_w}"/></geometry>
-        <material name="wheel_black"><color rgba="0.08 0.08 0.08 1.0"/></material>
+        <material name="wheel_rubber"><color rgba="0.22 0.20 0.17 1.0"/></material>
       </visual>
       <collision>
@@ -207,5 +207,13 @@
   <xacro:macro name="wheel_physics" params="link">
     <gazebo reference="${link}">
-      <material>Gazebo/Black</material>
+      <!-- 고무 타이어: 다크 챠콜 + 극저 specular(무광) + 약간 warm 브라운 톤 -->
+      <visual>
+        <material>
+          <ambient>0.12 0.11 0.09 1.0</ambient>
+          <diffuse>0.22 0.20 0.17 1.0</diffuse>
+          <specular>0.02 0.02 0.02 1.0</specular>
+          <emissive>0.0 0.0 0.0 1.0</emissive>
+        </material>
+      </visual>
       <mu1>1.0</mu1>
       <mu2>1.0</mu2>

Commit message: hardware rearrange

File: src/ackermann_car_description/urdf/ackermann_car.urdf.xacro (robot description, xacro)
@@ -12,5 +12,5 @@
   <xacro:property name="body_l"       value="0.440"/>
   <xacro:property name="body_w"       value="0.200"/>
-  <xacro:property name="body_h"       value="0.080"/>
+  <xacro:property name="body_h"       value="0.140"/>
   <xacro:property name="chassis_mass" value="1.5"/>
   <xacro:property name="wheel_mass"   value="0.1"/>
@@ -30,10 +30,10 @@
   <link name="base_link">
     <visual>
-      <origin xyz="0 0 0" rpy="0 0 0"/>
+      <origin xyz="0 0 0.03" rpy="0 0 0"/>
       <geometry><box size="${body_l} ${body_w} ${body_h}"/></geometry>
       <material name="chassis_blue"><color rgba="0.15 0.35 0.75 1.0"/></material>
     </visual>
     <collision>
-      <origin xyz="0 0 0" rpy="0 0 0"/>
+      <origin xyz="0 0 0.03" rpy="0 0 0"/>
       <geometry><box size="${body_l} ${body_w} ${body_h}"/></geometry>
     </collision>
@@ -165,5 +165,5 @@
     <parent link="base_link"/>
     <child  link="camera_link"/>
-    <origin xyz="${body_l/2 + 0.015} 0 0" rpy="0 0 0"/>
+    <origin xyz="${body_l/2 + 0.015} 0 0.10" rpy="0 0 0"/>
   </joint>
   <link name="camera_link">
